File: electrical/ReMapper/ReMapper.kicad_pcb (KiCad board)
At the start: 4 copper layers, 35 x 65 mm, 43 parts, among them J1 ESP_UART0, J2 I2C Display, J3 USB_IN, J4 USB_OUT, J5 Button GND Pad, J9 Button Socket, U1 SPX1117M3-L-3-3/TR, U2 W25Q128JVE, U3 ESP32-S3-WROOM-1-N8R8, U4 RP2040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

Commit message: working on fab
Parts:
- moved G*** 2.94 mm to (185.7, 76.5)
Changed lines of the file:
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@@
 	(footprint "LOGO"
 		(layer "F.Cu")
-		(at 184.4294 73.8378 90)
+		(at 185.72185 76.480422 90)
 		(property "Reference" "G***"
 			(at 0 0 90)
@@
 		)
 	)
-	(gr_text "ReMapper Rev4\nCedarHacks.com"
-		(at 182.0926 69.4436 90)
+	(gr_text "ReMapper\nRev4\nCedarHacks.com"
+		(at 183.496953 73.1012 90)
 		(layer "F.SilkS")
 		(effects
